Commit message: changed arm closer to setup

File: cartesian_controller_simulation/urdf/arm2.urdf.xacro (robot description, xacro)
@@ -3,17 +3,16 @@
         <!--
         RoboNav Arm URDF - 5 degrees of freedom
-        Modified to remove joint6/link6
+        joint 1 is prismatic along x axis (left-right motion)
+        joint 2,3,4 are revolute along y axis (pitch motion)
+        joint 5 is attached to joint 4 and is along x-axis (roll motion)
+        aka joint 4 and 5 form a wrist (pitch and roll)
         -->
         <xacro:include filename="$(find cartesian_controller_simulation)/urdf/joint.urdf.xacro"/>
         <!-- ROS2 control interfaces -->
         <ros2_control name="cartesian_controller_simulation" type="system">
-                <xacro:joint_interface name="joint1" p="1000" d="0.5" />
-                <xacro:joint_interface name="joint2" p="1000" d="0.5" />
-                <xacro:joint_interface name="joint3" p="500" d="0.5" />
-                <xacro:joint_interface name="joint4" p="100" d="0.5" />
-                <joint name="joint5">
+                <joint name="joint1"> //base slide - prismatic
                 <command_interface name="position">
-                        <param name="min">-0.2</param>
-                        <param name="max">0.2</param>
+                        <param name="min">-0.5</param>
+                        <param name="max">0.5</param>
                 </command_interface>
                 <command_interface name="velocity">
@@ -27,5 +26,8 @@
                 <state_interface name="effort"/>
                 </joint>
-                <!-- Removed joint6 interface -->
+                <xacro:joint_interface name="joint2" p="1000" d="0.5" /> //shoulder pitch
+                <xacro:joint_interface name="joint3" p="500" d="0.5" /> // elbow pitch
+                <xacro:joint_interface name="joint4" p="100" d="0.5" /> //wrist pitch
+                <xacro:joint_interface name="joint5" p="50" d="0.5" /> //wrist roll
                 <hardware>
                         <plugin>cartesian_controller_simulation/Simulator</plugin>
@@ -41,5 +43,5 @@
         <xacro:property name="link2_length" value="0.5" />
         <xacro:property name="link3_length" value="0.5" />
-        <xacro:property name="link4_length" value="0.15" />
+        <xacro:property name="link4_length" value="0.08" />
         <xacro:property name="link5_length" value="0.10" />
         <!-- Removed link6_length -->
@@ -93,10 +95,11 @@
                 </visual>
         </link>
-        <joint name="joint1" type="revolute"> // ask if continous or revolute
+        <!-- Prismatic slider -->
+        <joint name="joint1" type="prismatic"> // base slide
                 <parent link="base_link" />
                 <child link = "link1" />
                 <origin xyz="0.0 0.0 ${3.0 / 2.0 * joint_length}" rpy="0.0 0.0 0.0" />
-                <axis xyz="0 0 1" />
-                <limit lower="${-2.0 * pi}" upper="${2.0 * pi}" effort="1.0" velocity="10.0"/>
+                <axis xyz="1 0 0" />
+                <limit lower="-0.5" upper="0.5" effort="100" velocity="1.0"/>
         </joint>
         <link name="link1">
@@ -126,4 +129,5 @@
                 </visual>
         </link>
+        <!-- Shoulder pitch joint -->
         <joint name="joint2" type="revolute">
                 <parent link="link1" />
@@ -159,5 +163,6 @@
                 </visual>
         </link>
-        <joint name="joint3" type="revolute"> // ask if continous or revolute
+        <!-- Elbow pitch joint -->
+        <joint name="joint3" type="revolute"> //elbow pitch
                 <parent link="link2" />
                 <child link = "link3" />
@@ -192,4 +197,5 @@
                 </visual>
         </link>
+        <!-- Wrist pitch joint -->
         <joint name="joint4" type="revolute">
                 <parent link="link3" />
@@ -225,15 +231,16 @@
                 </visual>
         </link>
-        <joint name="joint5" type="prismatic">
+        <!-- Wrist roll joint -->
+        <joint name="joint5" type="revolute">
                 <parent link="link4" />
                 <child link = "link5" />
-                <origin xyz="0.0 ${link4_length} ${joint_length}" rpy="0.0 0.0 0.0" />
-                <axis xyz="0 0 1" />
-                <limit lower="-0.2" upper="0.2" effort="1.0" velocity="1.0"/>
+                <origin xyz="0.0 ${link4_length} 0" rpy="0.0 0.0 0.0" />
+                <axis xyz="0 1 0" />
+                <limit lower="${-pi}" upper="${pi}" effort="1.0" velocity="2.0"/>
         </joint>
         <link name="link5">
                 <inertial>
-                        <origin xyz="0 0 ${link5_length * 1.5}" rpy="0 0 0"/>
-                        <mass value="1"/>
+                        <origin xyz="0 ${link5_length * 1.5} 0" rpy="0 0 0"/>
+                        <mass value="0.5"/>
                         <inertia ixx="1.0"  ixy="0"  ixz="0" iyy="1.0" iyz="0" izz="1.0" />
                 </inertial>
@@ -246,5 +253,5 @@
                 </visual>
                 <visual name="link">
-                        <origin xyz="0 0 ${link5_length * 1.5}" rpy="0 0 0" />
+                        <origin xyz="0 ${link5_length * 1.5} 0" rpy="${pi/2.0} 0 0" />
                         <geometry>
                                 <cylinder length="${link5_length * 3}" radius="${link_radius * 1.5}"/>
@@ -257,5 +264,5 @@
         <!-- Attach a sensor link at the end of link5 -->
         <joint name="sensor_link_joint" type="fixed">
-                <origin xyz="0 0 ${link5_length * 3}" rpy="0 0 0"/>
+                <origin xyz="0 ${link5_length * 3} 0" rpy="0 0 0"/>
                 <parent link="link5"/>
                 <child link="sensor_link"/>

Commit message: Fix joint axis and dimensions in arm2 model for accurate simulation

File: cartesian_controller_simulation/urdf/arm2.urdf.xacro (robot description, xacro)
@@ -3,5 +3,5 @@
         <!--
         RoboNav Arm URDF - 5 degrees of freedom
-        joint 1 is prismatic along x axis (left-right motion)
+        joint 1 is prismatic along y axis (left-right motion)
         joint 2,3,4 are revolute along y axis (pitch motion)
         joint 5 is attached to joint 4 and is along x-axis (roll motion)
@@ -42,7 +42,7 @@
         <xacro:property name="link1_length" value="0.15" />
         <xacro:property name="link2_length" value="0.5" />
-        <xacro:property name="link3_length" value="0.5" />
-        <xacro:property name="link4_length" value="0.08" />
-        <xacro:property name="link5_length" value="0.10" />
+        <xacro:property name="link3_length" value="0.3" />
+        <xacro:property name="link4_length" value="0.1" />
+        <xacro:property name="link5_length" value="0.05" />
         <!-- Removed link6_length -->
         <!-- colors -->
@@ -100,5 +100,5 @@
                 <child link = "link1" />
                 <origin xyz="0.0 0.0 ${3.0 / 2.0 * joint_length}" rpy="0.0 0.0 0.0" />
-                <axis xyz="1 0 0" />
+                <axis xyz="0 1 0" />
                 <limit lower="-0.5" upper="0.5" effort="100" velocity="1.0"/>
         </joint>
@@ -201,5 +201,5 @@
                 <parent link="link3" />
                 <child link = "link4" />
-                <origin xyz="0.0 ${joint_length} ${link3_length}" rpy="0.0 ${pi / 2.0} 0.0" />
+                <origin xyz="0.0 ${joint_length} ${link3_length}" rpy="0.0 0.0 0.0" />
                 <axis xyz="0 1 0" />
                 <limit lower="${-2.0 * pi}" upper="${2.0 * pi}" effort="1.0" velocity="10.0"/>
@@ -212,5 +212,5 @@
                 </inertial>
                 <visual name="joint4">
-                        <origin xyz="0 0 0" rpy="${pi / 2.0} 0 0" />
+                        <origin xyz="0 0 0" rpy="0 0 0" />
                         <geometry>
                                 <cylinder length="${joint_length}" radius="${joint_radius}"/>
@@ -219,5 +219,5 @@
                 </visual>
                 <visual name="link">
-                        <origin xyz="0 ${link4_length / 2.0} 0" rpy="${pi / 2.0} 0 0" />
+                        <origin xyz="0 0 ${link4_length / 2.0}" rpy="0 0 0" />
                         <geometry>
                                 <cylinder length="${link4_length}" radius="${link_radius}"/>
@@ -225,5 +225,5 @@
                 </visual>
                 <visual name="joint5">
-                        <origin xyz="0 ${link4_length} 0" rpy="0 0 0" />
+                        <origin xyz="0 0 ${link4_length}" rpy="${pi / 2.0} 0 0" />
                         <geometry>
                                 <cylinder length="${joint_length}" radius="${joint_radius}"/>
@@ -235,5 +235,5 @@
                 <parent link="link4" />
                 <child link = "link5" />
-                <origin xyz="0.0 ${link4_length} 0" rpy="0.0 0.0 0.0" />
+                <origin xyz="0.0 0 ${link4_length}" rpy="0.0 ${pi / 2.0} 0.0" />
                 <axis xyz="0 1 0" />
                 <limit lower="${-pi}" upper="${pi}" effort="1.0" velocity="2.0"/>
@@ -241,5 +241,5 @@
         <link name="link5">
                 <inertial>
-                        <origin xyz="0 ${link5_length * 1.5} 0" rpy="0 0 0"/>
+                        <origin xyz="0 0 ${link5_length * 1.5}" rpy="0 0 0"/>
                         <mass value="0.5"/>
                         <inertia ixx="1.0"  ixy="0"  ixz="0" iyy="1.0" iyz="0" izz="1.0" />
@@ -253,5 +253,5 @@
                 </visual>
                 <visual name="link">
-                        <origin xyz="0 ${link5_length * 1.5} 0" rpy="${pi/2.0} 0 0" />
+                        <origin xyz="0 0 ${link5_length * 1.5}" rpy="0 0 0" />
                         <geometry>
                                 <cylinder length="${link5_length * 3}" radius="${link_radius * 1.5}"/>
@@ -264,5 +264,5 @@
         <!-- Attach a sensor link at the end of link5 -->
         <joint name="sensor_link_joint" type="fixed">
-                <origin xyz="0 ${link5_length * 3} 0" rpy="0 0 0"/>
+                <origin xyz="0 0 ${link5_length * 3}" rpy="0 0 0"/>
                 <parent link="link5"/>
                 <child link="sensor_link"/>
